File: hardware/_autosave-loeti.kicad_pcb (KiCad board)
At the start: 2 copper layers, 60 x 80 mm, 58 parts, among them J1 USB_C_Receptacle_USB2.0, J2 Samtec FTS-107-01-L-D, J3 AudioJack4, Q1 BC817, Q2 BC817, Q3 BC807, Q4 Si4825DDY, DMG4435SSS, IRF939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, SW1 key2, SW2 SW_SPST, SW3 SW_SPST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

Commit message: improved UI
Routing:
- net ADC_IN2: track 34.1 -> 48.3 mm, vias 1 -> 2
- net +3V3: track 54.2 -> 55.2 mm
Changed lines of the file:
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@@
     (thickness 1.6)
     (drawings 18)
-    (tracks 504)
+    (tracks 512)
     (zones 0)
     (modules 58)
@@
   (segment (start 85.65 57.975) (end 85.625 57.975) (width 0.15) (layer F.Cu) (net 1))
   (segment (start 85.625 57.975) (end 84.8 58.8) (width 0.15) (layer F.Cu) (net 1))
-  (via (at 84.8 50.5) (size 0.6) (drill 0.3) (layers F.Cu B.Cu) (net 1))
-  (segment (start 89.425 50.5) (end 91.225 48.7) (width 0.15) (layer F.Cu) (net 1))
-  (segment (start 84.8 50.5) (end 89.425 50.5) (width 0.15) (layer F.Cu) (net 1))
   (via (at 100 67.6) (size 0.6) (drill 0.3) (layers F.Cu B.Cu) (net 1))
   (segment (start 101.1 67.625) (end 100.025 67.625) (width 0.15) (layer F.Cu) (net 1))
@@
   (segment (start 84.675 48.1) (end 84.8 48.1) (width 0.15) (layer F.Cu) (net 1))
   (segment (start 84.8 45.55) (end 84.8 48.1) (width 0.15) (layer F.Cu) (net 1))
-  (segment (start 84.8 48.1) (end 84.8 50.5) (width 0.15) (layer F.Cu) (net 1))
   (via (at 104.75 69.95) (size 0.6) (drill 0.3) (layers F.Cu B.Cu) (net 1))
+  (segment (start 89.425 50.5) (end 91.225 48.7) (width 0.15) (layer F.Cu) (net 1))
+  (via (at 84.1 50.5) (size 0.6) (drill 0.3) (layers F.Cu B.Cu) (net 1))
+  (segment (start 84.1 50.5) (end 89.425 50.5) (width 0.15) (layer F.Cu) (net 1))
+  (segment (start 84.1 48.675) (end 84.1 50.5) (width 0.15) (layer F.Cu) (net 1))
+  (segment (start 84.675 48.1) (end 84.1 48.675) (width 0.15) (layer F.Cu) (net 1))
   (segment (start 81.1375 63.6) (end 81.1375 64.1) (width 0.15) (layer F.Cu) (net 2))
   (segment (start 77.8 63.6) (end 77.65 63.75) (width 0.15) (layer F.Cu) (net 2))
@@
   (segment (start 79.1 47.475) (end 79.4 47.175) (width 0.15) (layer F.Cu) (net 23))
   (segment (start 79.1 49.05) (end 79.1 47.475) (width 0.15) (layer F.Cu) (net 23))
+  (segment (start 79.1 49.05) (end 79.65 49.05) (width 0.15) (layer F.Cu) (net 23))
+  (via (at 80.2 48.5) (size 0.6) (drill 0.3) (layers F.Cu B.Cu) (net 23))
+  (segment (start 79.65 49.05) (end 80.2 48.5) (width 0.15) (layer F.Cu) (net 23))
+  (segment (start 80.2 48.5) (end 83 48.5) (width 0.15) (layer B.Cu) (net 23))
+  (segment (start 83 48.5) (end 84.2 49.7) (width 0.15) (layer B.Cu) (net 23))
+  (segment (start 84.2 49.7) (end 84.8 50.3) (width 0.15) (layer B.Cu) (net 23))
+  (segment (start 84.8 50.3) (end 84.8 57.9) (width 0.15) (layer B.Cu) (net 23))
   (via (at 98 72.3) (size 0.6) (drill 0.3) (layers F.Cu B.Cu) (net 24))
   (segment (start 96.675 72.3) (end 98 72.3) (width 0.15) (layer F.Cu) (net 24))
@@
     (polygon
       (pts
-        (xy 119 121.5) (xy 61 121.5) (xy 61 41.5) (xy 119 41.5)
+        (xy 118 121.5) (xy 62 121.5) (xy 62 41.5) (xy 118 41.5)
       )
     )
@@
     (polygon
       (pts
-        (xy 119 121.5) (xy 61 121.5) (xy 61 41.5) (xy 119 41.5)
+        (xy 118 121.5) (xy 62 121.5) (xy 62 41.5) (xy 118 41.5)
       )
     )
@@
     (polygon
       (pts
-        (xy 119 58.15) (xy 119 64) (xy 85.5 64) (xy 85.5 49.5) (xy 83.75 47.75)
-        (xy 83.75 63.25) (xy 61 63.25) (xy 61 41.5) (xy 119 41.5)
+        (xy 118 58.5) (xy 118 64) (xy 85.5 64) (xy 85.5 49.5) (xy 83.75 47.75)
+        (xy 83.75 63.25) (xy 62 63.25) (xy 62 41.5) (xy 118 41.5)
       )
     )
