File: hardware/loeti.sch (KiCad schematic (older format))
At the start: 63 parts, among them J1 USB_C_Receptacle_USB2.0, J2 20021112-00014T1LF, J3 AudioJack4, Q1 BC817, Q2 BC817, Q3 BC807, Q4 Si4825DDY, DMG4435SSS, IRF939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, SW1 key2, SW2 SW_SPST, SW3 SW_SPST, U1 AP2204R-3.3, U2 STUSB4500QTR, U3 USBLC6-2SC6, U4 EA_DOGS104B-A, U5 STM32F042K6Tx, U6 ADS1118IDGS, U7 INA138, U8 ASSR-1218, U9 ASSR-1218

Commit message: v4, stusb final
Parts:
- removed J3: AudioJack4, custom:CUI_SJ-43614-SMT, symbol Connector:AudioJack4
- removed U7: INA138, Package_TO_SOT_SMD:SOT-23-5, symbol Amplifier_Current:INA138
- added D4, D5: BAT54S, Package_TO_SOT_SMD:SOT-23, symbol Diode:BAT54S
- added J3: AudioJack3, custom:CUI_SJ-3502-SMT, symbol Connector:AudioJack3
- added R22: 10k, Resistor_SMD:R_0603_1608Metric_Pad1.05x0.95mm_HandSolder, symbol Device:R
- added U7: INA301A, Package_SO:VSSOP-8_3.0x3.0mm_P0.65mm, symbol custom:INA301
- R15: value WSL2010R0200FEA18 -> WSLP2010R0100FEA
- R16: value 100k -> 25k
Connections:
- net labels added: CUR_LIMIT, CUR_NALERT, CUR_RESET
- wire segments 223 -> 225
- no-connect marks 18 -> 17
Other:
- note added: "10 mOhm shunt\n20 V/V gain\n10 A in -> 2 V out"
- note added: "ESD protection for ADC inputs"
- moved on the sheet: C18, D1, D2, R11, R17, R18, R19, R6, R7, R9, SW1, SW2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

Commit message: v4 production version
Parts:
- removed R11, R9: 20, Resistor_SMD:R_0603_1608Metric_Pad1.05x0.95mm_HandSolder, symbol Device:R
- removed U3: USBLC6-2SC6, Package_TO_SOT_SMD:SOT-23-6, symbol Power_Protection:USBLC6-2SC6
- removed U5: STM32F042K6Tx, Package_QFP:LQFP-32_7x7mm_P0.8mm, symbol MCU_ST_STM32F0:STM32F042K6Tx
- added U5: STM32F030K6Tx, Package_QFP:LQFP-32_7x7mm_P0.8mm, symbol MCU_ST_STM32F0:STM32F030K6Tx
Connections:
- net +3V3: now also U5.1 (VDD), U5.17 (VDD), U5.5 (VDDA)
- net ADC_IN2: now also U5.8 (PA2)
- net ADC_IN7: now also U5.13 (PA7)
- net CUR_NALERT: now also U5.3 (PF1)
- net CUR_RESET: now also U5.2 (PF0)
- net GND: now also U5.16 (VSS), U5.32 (VSS)
- net I2C1_SCL: now also U5.29 (PB6)
- net I2C1_SDA: now also U5.30 (PB7)
- net LCD_NRST: now also U5.12 (PA6)
- net NRST: now also U5.4 (NRST)
- net PD_ALERT_INT: now also U5.21 (PA11)
- net PD_RST: now also U5.15 (PB1)
- net PWM: now also U5.18 (PA8)
- net SEL_TC_0: now also U5.10 (PA4)
- net SEL_TC_1: now also U5.9 (PA3)
- net SPI1_MISO: now also U5.27 (PB4)
- net SPI1_MOSI: now also U5.28 (PB5)
- net SPI1_NSS1: now also U5.25 (PA15)
- net SPI1_NSS2: now also U5.22 (PA12)
- net SPI1_SCK: now also U5.26 (PB3)
- net SWCLK: now also U5.24 (PA14)
- net SWDIO: now also U5.23 (PA13)
- net at J1.A6 (D+): no longer J1.B6 (D+)
- net at J1.A7 (D-): no longer J1.B7 (D-)
- net BOOT0: now reaches R7.2
- net BOOT0: now also U5.31 (BOOT0)
- net VCP_RX: now reaches J2.13 (T_VCP_RX)
- net VCP_RX: now also U5.19 (PA9)
- net VCP_TX: now reaches J2.14 (VCP_TX)
- net VCP_TX: now also U5.20 (PA10)
- net at SW2.1 (A): now also U5.6 (PA0)
- net at SW3.1 (A): now also U5.7 (PA1)
- no-connect marks 17 -> 19
Other:
- moved on the sheet: R6, R7, SW1
Changed lines of the file:
@@
 Connection ~ 2350 8950
 Wire Wire Line
-	6050 3150 6050 3250
+	5950 3150 5950 3250
 Wire Wire Line
 	7150 4500 7150 4600
@@
 L power:GND #PWR024
 U 1 1 5A9ADA03
-P 6050 3250
-F 0 "#PWR024" H 6050 3000 50  0001 C CNN
-F 1 "GND" H 6055 3077 50  0000 C CNN
-F 2 "" H 6050 3250 50  0001 C CNN
-F 3 "" H 6050 3250 50  0001 C CNN
-	1    6050 3250
+P 5950 3250
+F 0 "#PWR024" H 5950 3000 50  0001 C CNN
+F 1 "GND" H 5955 3077 50  0000 C CNN
+F 2 "" H 5950 3250 50  0001 C CNN
+F 3 "" H 5950 3250 50  0001 C CNN
+	1    5950 3250
 	1    0    0    -1
 $EndComp
@@
 L Switch:SW_Push SW1
 U 1 1 5C1295B7
-P 6050 2950
-F 0 "SW1" V 6004 3098 50  0000 L CNN
-F 1 "key2" V 6095 3098 50  0000 L CNN
-F 2 "Button_Switch_SMD:SW_SPST_PTS810" H 6050 3150 50  0001 C CNN
-F 3 "" H 6050 3150 50  0001 C CNN
-	1    6050 2950
+P 5950 2950
+F 0 "SW1" V 5904 3098 50  0000 L CNN
+F 1 "key2" V 5995 3098 50  0000 L CNN
+F 2 "Button_Switch_SMD:SW_SPST_PTS810" H 5950 3150 50  0001 C CNN
+F 3 "" H 5950 3150 50  0001 C CNN
+	1    5950 2950
 	0    -1   1    0
 $EndComp
@@
 L power:+3V3 #PWR023
 U 1 1 5C1295BE
-P 6050 2250
-F 0 "#PWR023" H 6050 2100 50  0001 C CNN
-F 1 "+3V3" H 6065 2423 50  0000 C CNN
-F 2 "" H 6050 2250 50  0001 C CNN
-F 3 "" H 6050 2250 50  0001 C CNN
-	1    6050 2250
+P 5950 2250
+F 0 "#PWR023" H 5950 2100 50  0001 C CNN
+F 1 "+3V3" H 5965 2423 50  0000 C CNN
+F 2 "" H 5950 2250 50  0001 C CNN
+F 3 "" H 5950 2250 50  0001 C CNN
+	1    5950 2250
 	-1   0    0    -1
 $EndComp
 Wire Wire Line
-	6050 2250 6050 2350
+	5950 2250 5950 2350
 Wire Wire Line
 	2600 1900 2450 1900
@@
 Wire Wire Line
 	1850 3400 1850 3500
-Text GLabel 8850 3900 2    50   Input ~ 0
-USB_P
-Text GLabel 8850 3800 2    50   Input ~ 0
-USB_N
 $Comp
 L Device:C C9
@@
 	1    0    0    -1
 $EndComp
-Text GLabel 6750 3700 0    50   Input ~ 0
+Text GLabel 6650 3800 0    50   Input ~ 0
 SPI1_SCK
-Text GLabel 6750 3900 0    50   Input ~ 0
+Text GLabel 6650 4000 0    50   Input ~ 0
 SPI1_MOSI
 Text GLabel 7750 4200 2    50   Input ~ 0
 SPI1_NSS1
-Text GLabel 6750 3800 0    50   Input ~ 0
+Text GLabel 6650 3900 0    50   Input ~ 0
 SPI1_MISO
 Text GLabel 12100 2400 0    50   Input ~ 0
@@
 Text GLabel 15150 4800 2    50   Input ~ 0
 SPI1_MISO
-Text GLabel 7750 3700 2    50   Input ~ 0
+Text GLabel 7750 3900 2    50   Input ~ 0
 SPI1_NSS2
-Text GLabel 6750 4000 0    50   Input ~ 0
+Text GLabel 6650 4100 0    50   Input ~ 0
 I2C1_SCL
-Text GLabel 6750 4100 0    50   Input ~ 0
+Text GLabel 6650 4200 0    50   Input ~ 0
 I2C1_SDA
 Text GLabel 3700 7900 2    50   Input ~ 0
@@
 Text GLabel 3700 8100 2    50   Input ~ 0
 PD_ALERT_INT
-Text GLabel 7750 3600 2    50   Input ~ 0
+Text GLabel 7750 3800 2    50   Input ~ 0
 PD_ALERT_INT
 Wire Wire Line
-	6500 4650 6500 4750
+	8250 7100 8250 7200
 $Comp
 L power:GND #PWR026
 U 1 1 5E8122BA
-P 6500 4750
-F 0 "#PWR026" H 6500 4500 50  0001 C CNN
-F 1 "GND" H 6505 4577 50  0000 C CNN
-F 2 "" H 6500 4750 50  0001 C CNN
-F 3 "" H 6500 4750 50  0001 C CNN
-	1    6500 4750
-	1    0    0    -1
-$EndComp
-Wire Wire Line
-	6750 4200 6500 4200
-Wire Wire Line
-	6500 4200 6500 4350
+P 8250 7200
+F 0 "#PWR026" H 8250 6950 50  0001 C CNN
+F 1 "GND" H 8255 7027 50  0000 C CNN
+F 2 "" H 8250 7200 50  0001 C CNN
+F 3 "" H 8250 7200 50  0001 C CNN
+	1    8250 7200
+	1    0    0    -1
+$EndComp
+Wire Wire Line
+	8250 6650 8250 6800
 Text GLabel 14500 9200 2    50   Input ~ 0
 SHUNT-
@@
 L Device:R R6
 U 1 1 5E824254
-P 6050 2500
-F 0 "R6" H 5980 2454 50  0000 R CNN
-F 1 "10k" H 5980 2545 50  0000 R CNN
-F 2 "Resistor_SMD:R_0603_1608Metric_Pad1.05x0.95mm_HandSolder" V 5980 2500 50  0001 C CNN
-F 3 "~" H 6050 2500 50  0001 C CNN
-	1    6050 2500
+P 5950 2500
+F 0 "R6" H 5880 2454 50  0000 R CNN
+F 1 "10k" H 5880 2545 50  0000 R CNN
+F 2 "Resistor_SMD:R_0603_1608Metric_Pad1.05x0.95mm_HandSolder" V 5880 2500 50  0001 C CNN
+F 3 "~" H 5950 2500 50  0001 C CNN
+	1    5950 2500
 	1    0    0    -1
 $EndComp
@@
 L Device:R R7
 U 1 1 5E825484
-P 6500 4500
-F 0 "R7" H 6430 4454 50  0000 R CNN
-F 1 "10k" H 6430 4545 50  0000 R CNN
-F 2 "Resistor_SMD:R_0603_1608Metric_Pad1.05x0.95mm_HandSolder" V 6430 4500 50  0001 C CNN
-F 3 "~" H 6500 4500 50  0001 C CNN
-	1    6500 4500
+P 8250 6950
+F 0 "R7" H 8180 6904 50  0000 R CNN
+F 1 "10k" H 8180 6995 50  0000 R CNN
+F 2 "Resistor_SMD:R_0603_1608Metric_Pad1.05x0.95mm_HandSolder" V 8180 6950 50  0001 C CNN
+F 3 "~" H 8250 6950 50  0001 C CNN
+	1    8250 6950
 	-1   0    0    1
 $EndComp
@@
 Connection ~ 5800 7150
 NoConn ~ 5900 7250
-NoConn ~ 5900 7450
-NoConn ~ 7000 7450
 NoConn ~ 7000 7250
 Text GLabel 7000 6950 2    50   Input ~ 0
@@
 Text GLabel 7000 7350 2    50   Input ~ 0
 NRST
-Text GLabel 5650 2700 0    50   Input ~ 0
+Text GLabel 5550 2700 0    50   Input ~ 0
 NRST
 Text GLabel 7750 4000 2    50   Input ~ 0
@@
 Wire Wire Line
 	1500 4650 1500 4750
-Text GLabel 6750 3600 0    50   Input ~ 0
+Text GLabel 6650 3700 0    50   Input ~ 0
 PD_RST
 Wire Wire Line
@@
 $EndComp
 Wire Wire Line
-	5650 2700 6050 2700
-Wire Wire Line
-	6050 2650 6050 2700
-Connection ~ 6050 2700
-Wire Wire Line
-	6050 2700 6750 2700
-Wire Wire Line
-	6050 2700 6050 2750
-Text GLabel 4050 3050 2    50   Input ~ 0
-USB_P
-Text GLabel 4050 2050 2    50   Input ~ 0
-USB_N
-$Comp
-L Power_Protection:USBLC6-2SC6 U3
-U 1 1 5E962D2B
-P 3750 2550
-F 0 "U3" H 3750 3231 50  0000 C CNN
-F 1 "USBLC6-2SC6" H 3750 3140 50  0000 C CNN
-F 2 "Package_TO_SOT_SMD:SOT-23-6" H 3000 2950 50  0001 C CNN
-F 3 "http://www2.st.com/resource/en/datasheet/CD00050750.pdf" H 3950 2900 50  0001 C CNN
-	1    3750 2550
-	0    -1   -1   0
-$EndComp
-Wire Wire Line
-	2450 2400 2450 2500
-Wire Wire Line
-	2450 2600 2450 2700
-Wire Wire Line
-	3850 2050 4050 2050
-Wire Wire Line
-	3850 3050 4050 3050
-Wire Wire Line
-	3650 3050 3250 3050
-Wire Wire Line
-	3250 3050 3250 2700
-Wire Wire Line
-	3250 2700 2450 2700
-Connection ~ 2450 2700
-Wire Wire Line
-	2450 2400 3250 2400
-Wire Wire Line
-	3250 2400 3250 2050
-Wire Wire Line
-	3250 2050 3650 2050
-Connection ~ 2450 2400
-Wire Wire Line
-	2900 2550 3250 2550
-$Comp
-L power:GND #PWR019
-U 1 1 5E9A5EA0
-P 4250 2550
-F 0 "#PWR019" H 4250 2300 50  0001 C CNN
-F 1 "GND" H 4250 2400 50  0000 C CNN
-F 2 "" H 4250 2550 50  0001 C CNN
-F 3 "" H 4250 2550 50  0001 C CNN
-	1    4250 2550
-	0    -1   -1   0
-$EndComp
+	5550 2700 5950 2700
+Wire Wire Line
+	5950 2650 5950 2700
+Connection ~ 5950 2700
+Wire Wire Line
+	5950 2700 5950 2750
 $Comp
 L Device:D_Schottky_x2_ACom_KKA D1
@@
 Wire Wire Line
 	3750 4850 3850 4850
-$Comp
-L power:+3V3 #PWR011
-U 1 1 5E9E2C0E
-P 2900 2550
-F 0 "#PWR011" H 2900 2400 50  0001 C CNN
-F 1 "+3V3" H 2915 2723 50  0000 C CNN
-F 2 "" H 2900 2550 50  0001 C CNN
-F 3 "" H 2900 2550 50  0001 C CNN
-	1    2900 2550
-	0    -1   -1   0
-$EndComp
 $Comp
 L power:GND #PWR015
@@
 SWO
 $Comp
-L Device:R R9
-U 1 1 5ED7E821
-P 8300 3800
-F 0 "R9" H 8230 3754 50  0000 R CNN
-F 1 "20" H 8230 3845 50  0000 R CNN
-F 2 "Resistor_SMD:R_0603_1608Metric_Pad1.05x0.95mm_HandSolder" V 8230 3800 50  0001 C CNN
-F 3 "~" H 8300 3800 50  0001 C CNN
-	1    8300 3800
-	0    -1   -1   0
-$EndComp
-$Comp
-L Device:R R11
-U 1 1 5ED7F80E
-P 8600 3900
-F 0 "R11" H 8530 3854 50  0000 R CNN
-F 1 "20" H 8530 3945 50  0000 R CNN
-F 2 "Resistor_SMD:R_0603_1608Metric_Pad1.05x0.95mm_HandSolder" V 8530 3900 50  0001 C CNN
-F 3 "~" H 8600 3900 50  0001 C CNN
-	1    8600 3900
-	0    -1   -1   0
-$EndComp
-Wire Wire Line
-	8850 3800 8450 3800
-Wire Wire Line
-	8150 3800 7750 3800
-Wire Wire Line
-	7750 3900 8450 3900
-Wire Wire Line
-	8750 3900 8850 3900
-$Comp
 L Relay_SolidState:ASSR-1218 U8
 U 1 1 5EDBD456
@@
 Text GLabel 13450 9050 0    50   Input ~ 0
 CUR_LIMIT
-Text GLabel 6750 3300 0    50   Input ~ 0
+Text GLabel 6650 3400 0    50   Input ~ 0
 CUR_NALERT
-Text GLabel 6750 3200 0    50   Input ~ 0
+Text GLabel 6650 3300 0    50   Input ~ 0
 CUR_RESET
-$Comp
-L MCU_ST_STM32F0:STM32F042K6Tx U5
-U 1 1 5EAA038A
-P 7250 3400
-F 0 "U5" H 7250 2311 50  0000 C CNN
-F 1 "STM32F042K6Tx" H 7250 2220 50  0000 C CNN
-F 2 "Package_QFP:LQFP-32_7x7mm_P0.8mm" H 6850 2500 50  0001 R CNN
-F 3 "http://www.st.com/st-web-ui/static/active/en/resource/technical/document/datasheet/DM00105814.pdf" H 7250 3400 50  0001 C CNN
-	1    7250 3400
-	1    0    0    -1
-$EndComp
 Text GLabel 8050 5900 0    50   Input ~ 0
 ADC_IN2
@@
 Wire Wire Line
 	5900 8800 6000 8800
-NoConn ~ 6750 3500
-NoConn ~ 7750 3200
 Text GLabel 11350 8750 0    50   Input ~ 0
 CUR_NALERT
@@
 Text Notes 14200 8500 0    50   ~ 0
 10 mOhm shunt\n20 V/V gain\n10 A in -> 2 V out
+$Comp
+L MCU_ST_STM32F0:STM32F030K6Tx U5
+U 1 1 5EDA1F44
+P 7250 3400
+F 0 "U5" H 7200 2311 50  0000 C CNN
+F 1 "STM32F030K6Tx" H 7200 2220 50  0000 C CNN
+F 2 "Package_QFP:LQFP-32_7x7mm_P0.8mm" H 6750 2500 50  0001 R CNN
+F 3 "http://www.st.com/st-web-ui/static/active/en/resource/technical/document/datasheet/DM00088500.pdf" H 7250 3400 50  0001 C CNN
+	1    7250 3400
+	1    0    0    -1
+$EndComp
+Wire Wire Line
+	8250 6650 8600 6650
+NoConn ~ 2450 2400
+NoConn ~ 2450 2500
+NoConn ~ 2450 2600
+NoConn ~ 2450 2700
+Wire Wire Line
+	6650 2700 5950 2700
+Text GLabel 6650 2900 0    50   Input ~ 0
+BOOT0
+Text GLabel 8600 6650 2    50   Input ~ 0
+BOOT0
+Text GLabel 7000 7450 2    50   Input ~ 0
+VCP_TX
+Text GLabel 5900 7450 0    50   Input ~ 0
+VCP_RX
+Text GLabel 7750 3600 2    50   Input ~ 0
+VCP_RX
+Text GLabel 7750 3700 2    50   Input ~ 0
+VCP_TX
+NoConn ~ 6650 3600
+NoConn ~ 7750 3200
 $EndSCHEMATC

Commit message: preliminary layout
Parts:
- removed C10: 1μF 25V, Capacitor_SMD:C_0603_1608Metric_Pad1.05x0.95mm_HandSolder, symbol Device:C
- removed C13, C16, C18, C19: 0.1μF, Capacitor_SMD:C_0603_1608Metric_Pad1.05x0.95mm_HandSolder, symbol Device:C
- removed C17: EEU-FR1V471L, custom:CP_Radial_D8.0mm_P3.50mm_HOR, symbol Device:CP
- removed C2: 4.7μF 25V, Capacitor_SMD:C_0805_2012Metric_Pad1.15x1.40mm_HandSolder, symbol Device:C
- removed D5: BAT54S, Package_TO_SOT_SMD:SOT-23, symbol Diode:BAT54S
- removed J3: AudioJack3, custom:CUI_SJ-3502-SMT, symbol Connector:AudioJack3
- removed R17, R19, R22: 10k, Resistor_SMD:R_0603_1608Metric_Pad1.05x0.95mm_HandSolder, symbol Device:R
- removed R18: 1k, Resistor_SMD:R_0603_1608Metric_Pad1.05x0.95mm_HandSolder, symbol Device:R
- removed R20, R21: 470, Resistor_SMD:R_0603_1608Metric_Pad1.05x0.95mm_HandSolder, symbol Device:R
- removed R8: 1M, Resistor_SMD:R_0603_1608Metric_Pad1.05x0.95mm_HandSolder, symbol Device:R
- removed SW1: key2, Button_Switch_SMD:SW_SPST_PTS810, symbol Switch:SW_Push
- removed SW2, SW3: SW_SPST, custom:Omron-B3AL, symbol Switch:SW_SPST
- removed TP2: GND, TestPoint:TestPoint_THTPad_4.0x4.0mm_Drill2.0mm, symbol Connector:TestPoint
- removed TP3: 3V3, TestPoint:TestPoint_THTPad_4.0x4.0mm_Drill2.0mm, symbol Connector:TestPoint
- removed U4: EA_DOGS104B-A, Display:EA_DOGS104X-A, symbol Display_Graphic:EA_DOGS104B-A
- removed U6: ADS1118IDGS, Package_SO:VSSOP-10_3x3mm_P0.5mm, symbol Analog_ADC:ADS1118IDGS
- removed U7: INA301A, Package_SO:VSSOP-8_3.0x3.0mm_P0.65mm, symbol custom:INA301
- removed U8, U9: ASSR-1218, Package_SO:SO-4_4.4x4.3mm_P2.54mm, symbol Relay_SolidState:ASSR-1218
- added C11, C5: 1μF 25V, Capacitor_SMD:C_0805_2012Metric_Pad1.18x1.45mm_HandSolder, symbol Device:C
- added C13, C16: CP, Capacitor_SMD:CP_Elec_6.3x5.9, symbol Device:CP
- added C15, C17: 0.1μF, Capacitor_SMD:C_0603_1608Metric_Pad1.08x0.95mm_HandSolder, symbol Device:C
- added D4, D6, D7: LED, LED_THT:LED_D3.0mm, symbol Device:LED
- added J2: AudioJack3, custom:CUI_SJ-3502-SMT, symbol Connector:AudioJack3
- added R11, R14, R15: 1k, Resistor_SMD:R_0603_1608Metric_Pad0.98x0.95mm_HandSolder, symbol Device:R
- added SW1: D6R, custom:D6R, symbol custom:D6R
- added U4: TLV333-DBV, Package_TO_SOT_SMD:SOT-23-5_HandSoldering, symbol custom:TLV333-DBV
- added U5: INA239, Package_SO:VSSOP-10_3x3mm_P0.5mm, symbol custom:INA239
- C1, C14: footprint Capacitor_SMD:C_0603_1608Metric_Pad1.05x0.95mm_HandSolder -> Capacitor_SMD:C_0805_2012Metric_Pad1.18x1.45mm_HandSolder
- C10: renamed from C11; footprint Capacitor_SMD:C_0603_1608Metric_Pad1.05x0.95mm_HandSolder -> Capacitor_SMD:C_0805_2012Metric_Pad1.18x1.45mm_HandSolder
- C12: value 1μF 25V -> 0.1μF; footprint Capacitor_SMD:C_0603_1608Metric_Pad1.05x0.95mm_HandSolder -> Capacitor_SMD:C_0603_1608Metric_Pad1.08x0.95mm_HandSolder
- C2: renamed from C3; footprint Capacitor_SMD:C_0603_1608Metric_Pad1.05x0.95mm_HandSolder -> Capacitor_SMD:C_0805_2012Metric_Pad1.18x1.45mm_HandSolder
- C3: renamed from C4; footprint Capacitor_SMD:C_0603_1608Metric_Pad1.05x0.95mm_HandSolder -> Capacitor_SMD:C_0805_2012Metric_Pad1.18x1.45mm_HandSolder
- C4: renamed from C5; footprint Capacitor_SMD:C_0603_1608Metric_Pad1.05x0.95mm_HandSolder -> Capacitor_SMD:C_0805_2012Metric_Pad1.18x1.45mm_HandSolder
- C6, C7, C8, C9: footprint Capacitor_SMD:C_0603_1608Metric_Pad1.05x0.95mm_HandSolder -> Capacitor_SMD:C_0603_1608Metric_Pad1.08x0.95mm_HandSolder
- J1: footprint custom:CX90M-16P -> Connector_USB:USB_C_Receptacle_GCT_USB4085; symbol Connector:USB_C_Receptacle_USB2.0 -> loeti-rescue:USB_C_Receptacle_USB2.0-Connector
- R1, R2, R3, R4, R5, R6, R7: footprint Resistor_SMD:R_0603_1608Metric_Pad1.05x0.95mm_HandSolder -> Resistor_SMD:R_0603_1608Metric_Pad0.98x0.95mm_HandSolder
- R10: value 47 -> 220k; footprint Resistor_SMD:R_0603_1608Metric_Pad1.05x0.95mm_HandSolder -> Resistor_SMD:R_0603_1608Metric_Pad0.98x0.95mm_HandSolder
- R12: renamed from R14; footprint Resistor_SMD:R_0603_1608Metric_Pad1.05x0.95mm_HandSolder -> Resistor_SMD:R_0603_1608Metric_Pad0.98x0.95mm_HandSolder
- R13: renamed from R15; footprint Resistor_SMD:R_2010_5025Metric_Pad1.52x2.65mm_HandSolder -> Resistor_SMD:R_2010_5025Metric_Pad1.40x2.65mm_HandSolder
- R16: value 25k -> 1k; footprint Resistor_SMD:R_0603_1608Metric_Pad1.05x0.95mm_HandSolder -> Resistor_SMD:R_0603_1608Metric_Pad0.98x0.95mm_HandSolder
- R8: renamed from R12; footprint Resistor_SMD:R_0603_1608Metric_Pad1.05x0.95mm_HandSolder -> Resistor_SMD:R_0603_1608Metric_Pad0.98x0.95mm_HandSolder
- R9: renamed from R13; footprint Resistor_SMD:R_0603_1608Metric_Pad1.05x0.95mm_HandSolder -> Resistor_SMD:R_0603_1608Metric_Pad0.98x0.95mm_HandSolder
- renumbered D4 to D3, D3 to D5, J2 to J3, U5 to U3
Connections:
- net CUR_LIMIT is gone; now on net LED2: R16.2
- net +3V3: now also C14.1, C17.1, U4.5 (V+), U5.6 (VS); no longer C12.1
- net ADC_IN2: now also C12.1, R10.1, U4.1
- net GND: now also C14.2, C11.2, C13.2, C15.2, C16.2, C17.2, C5.2, D4.1 (K), D6.1 (K), D7.1 (K), J2.S, R11.2, SW1.3 (B), SW1.4 (B), U4.2 (V-), U5.7 (GND); no longer C12.2, C14.1, R16.1
- net HEATER+: now also J2.T
- net PWM: now also U3.14 (PB0); no longer U3.18 (PA8)
- net SPI1_MISO: now also U5.2 (MOSI)
- net SPI1_MOSI: now also U5.4 (MISO)
- net SPI1_SCK: now also U5.5 (SCLK)
- net T+: now also C15.1, J2.R, U4.3 (+)
- net VBUS: now also C11.1, C5.1, U5.10 (+), U5.8 (VBUS); no longer Q2.3 (C), R9.2
- net VCP_RX: now also U3.20 (PA10); no longer U3.19 (PA9)
- net VCP_TX: now also U3.19 (PA9); no longer U3.20 (PA10)
- net at R10.2: now also C12.2, R11.1, U4.4 (-); no longer C14.2
- net LED2: now reaches U3.11 (PA5)
- net ADC_IN7: no longer names the net of U3.13 (PA7)
- net CUR_NALERT renamed CURR_ALERT
- net CURR_ALERT: now also U5.3 (ALERT)
- net CUR_RESET renamed CURR_CS
- net CURR_CS: now also U5.1 (nCS)
- net LCD_NRST: no longer names the net of U3.12 (PA6)
- net SEL_TC_0 renamed LED1
- net LED1: now also R15.2
- net SEL_TC_1 renamed LED0
- net LED0: now also R14.2
- net SHUNT- renamed VPP
- net VPP: now also Q2.3 (C), R9.2, C13.1, C16.1, U5.9 (-)
- net SPI1_NSS1 renamed SW
- net SW: now also SW1.1 (A), SW1.2 (A)
- new net: D4.2 (A), R14.1
- new net: D6.2 (A), R15.1
- new net: D7.2 (A), R16.1
- no-connect marks 19 -> 15
Other:
- note added: "10 mOhm shunt"
- note added: "Connector"
- note added: "ESD protection for ADC input"
- note added: "UI"
- note removed: "10 mOhm shunt\n20 V/V gain\n10 A in -> 2 V out"
- note removed: "159 Hz low-pass"
- note removed: "1690 Hz low Pass"
- note removed: "Connectors and test points"
- note removed: "ESD protection for ADC inputs"
- note removed: "LCD"
- moved on the sheet: C1, C4, D1, D2, D3, R13, U1
