File: hardware/loeti.sch (KiCad schematic (older format))
At the start: 62 parts, among them J1 GCT USB4105, J2 AudioJack3, J3 20021112-00014T1LF, Q1 BC817, Q2 BC817, Q3 BC807, Q4 Si4825DDY, DMG4435SSS, IRF939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, SW1 D6R, U1 STUSB4500QTR, U2 AP2204R-3.3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

Commit message: initiali loeti tiny
Parts:
- C10, C11, C12, C13, C14, C6, C8, C9: footprint Capacitor_SMD:C_0603_1608Metric_Pad1.08x0.95mm_HandSolder -> Capacitor_SMD:C_0603_1608Metric
- C3, C4, C5, C7: footprint Capacitor_SMD:C_0805_2012Metric_Pad1.18x1.45mm_HandSolder -> Capacitor_SMD:C_0805_2012Metric
- D1, D3, D4, D8, D9: footprint Package_TO_SOT_SMD:SOT-323_SC-70_Handsoldering -> Package_TO_SOT_SMD:SOT-323_SC-70
- D11: footprint Package_TO_SOT_SMD:TSOT-23_HandSoldering -> Package_TO_SOT_SMD:TSOT-23
- D2: footprint Diode_SMD:D_0603_1608Metric_Pad1.05x0.95mm_HandSolder -> Diode_SMD:D_0603_1608Metric
- Q1, Q2, Q3: footprint Package_TO_SOT_SMD:SOT-23_Handsoldering -> Package_TO_SOT_SMD:SOT-23
- R1, R10, R11, R13, R14, R15, R16, R17, R18, R2, R21, R22, R23, R24, R3, R4, R5, R6, R7, R8, R9: footprint Resistor_SMD:R_0603_1608Metric_Pad0.98x0.95mm_HandSolder -> Resistor_SMD:R_0603_1608Metric
- R19: footprint Resistor_SMD:R_2010_5025Metric_Pad1.40x2.65mm_HandSolder -> Resistor_SMD:R_2010_5025Metric
- R20: value 20 -> 0.47; footprint Resistor_SMD:R_0603_1608Metric_Pad0.98x0.95mm_HandSolder -> Resistor_SMD:R_0603_1608Metric
- U2: footprint Package_TO_SOT_SMD:SOT-89-3_Handsoldering -> Package_TO_SOT_SMD:SOT-89-3
- U3: footprint Package_QFP:LQFP-32_7x7mm_P0.8mm -> Package_DFN_QFN:QFN-32-1EP_5x5mm_P0.5mm_EP3.1x3.1mm
- U4: footprint Package_TO_SOT_SMD:SOT-353_SC-70-5_Handsoldering -> Package_TO_SOT_SMD:SOT-353_SC-70-5
- U6: footprint Package_TO_SOT_SMD:SOT-23-6_Handsoldering -> Package_TO_SOT_SMD:SOT-23-6
- U7: footprint Package_TO_SOT_SMD:SOT-23-5_HandSoldering -> Package_TO_SOT_SMD:SOT-23-5
