File: hardware/loeti.kicad_sch (KiCad schematic)
At the start: 94 parts, among them J1 REDFIT_SWD_6, J2 AudioJack3, J3 USB_C_Receptacle_USB2.0, Q1 BC817, Q2 BC817, Q3 BC807, Q4 Si4425FDY, Q6 FDS6630A, SW1 RotaryEncoder_Switch, SW2 BOOT, U1 STM32G431C_6-8-B_Tx, U10 M24C64-RMN, U2 EA_OLEDS102-6, U3 USBLC6-2SC6, U4 74AHC1G08, U5 INA301, U6 Opamp_Dual, U8 AMS1117-3.3, X2 SG-210STF (16 MHz)

Commit message: feat: initial display implementation
Parts:
- removed U1: STM32G431C_6-8-B_Tx, Package_QFP:LQFP-48_7x7mm_P0.5mm, symbol MCU_ST_STM32G4:STM32G431C_6-8-B_Tx
- added U4: STM32G431CBTx, Package_QFP:LQFP-48_7x7mm_P0.5mm, symbol MCU_ST_STM32G4:STM32G431CBTx
- renumbered C28 to C1, C20 to C10, C29 to C11, C27 to C12, C1 to C13, C22 to C14, C23 to C15, C24 to C16, C25 to C17, C26 to C18, C3 to C19, C7 to C2, C4 to C20, C30 to C21, C31 to C22, C32 to C23, C21 to C24, C12 to C25, C13 to C26, C2 to C27, C16 to C28, C8 to C29, C15 to C3, C14 to C30, C10 to C31, C11 to C32, C5 to C4, C6 to C5, C9 to C6, C17 to C7, C18 to C8, C19 to C9, D3 to D1, D6 to D2, D7 to D3, D5 to D4, D2 to D5, D4 to D6, D10 to D7, D1 to D8, J3 to J2, J2 to J3, Q2 to Q1, Q6 to Q2, Q4 to Q3, Q1 to Q4, Q3 to Q5, R10 to R1, R30 to R10, R31 to R11, R32 to R12, R28 to R13, R33 to R14, R29 to R15, R18 to R16, R20 to R17, R15 to R18, R16 to R19, R1 to R2, R23 to R20, R17 to R21, R21 to R22, R9 to R23, R27 to R24, R22 to R25, R11 to R26, R25 to R27, R19 to R28, R13 to R29, R2 to R3, R24 to R30, R4 to R31, R14 to R32, R26 to R33, R8 to R4, R3 to R6, R12 to R7, R6 to R8, R7 to R9, SW2 to SW1, SW1 to SW2, U3 to U1, U10 to U3, U8 to U5, U4 to U6, U6 to U7, U7 to U8, U5 to U9, X2 to X1
Connections:
- net +3V3: now also U4.1 (VBAT), U4.21 (VDDA), U4.24 (VDD), U4.36 (VDD), U4.48 (VDD)
- net ADC2_IN3: now also U4.14 (PA6)
- net BOOT0: now also U4.45 (PB8)
- net CURR_ALERT: now also U4.22 (PB10)
- net CURR_RESET: now also U4.30 (PA8)
- net DAC1_OUT1: now also U4.12 (PA4)
- net GND: now also U4.19 (VSSA), U4.23 (VSS), U4.35 (VSS), U4.47 (VSS)
- net I2C1_SCL: now also U4.39 (PA15)
- net I2C1_SDA: now also U4.44 (PB7)
- net NRST: now also U4.7 (PG10)
- net OLED_D_C: now also U4.32 (PA10)
- net OLED_NRST: now also U4.31 (PA9)
- net ROT_A: now also U4.10 (PA2)
- net ROT_B: now also U4.11 (PA3)
- net ROT_SW: now also U4.9 (PA1)
- net SPI2_MISO: now also U4.28 (PB14)
- net SPI2_MOSI: now also U4.29 (PB15)
- net SPI2_NSS: now also U4.26 (PB12)
- net SPI2_SCK: now also U4.27 (PB13)
- net SWO: now also U4.40 (PB3)
- net TCK: now also U4.38 (PA14)
- net TIM2_CH4: now also U4.25 (PB11)
- net TMS: now also U4.37 (PA13)
- net UCPD_CC1: now also U4.43 (PB6)
- net UCPD_CC2: now also U4.41 (PB4)
- net USB_D_N: now also U4.33 (PA11)
- net USB_D_P: now also U4.34 (PA12)
- net at D1.3 (COM), R1.2: now also U4.8 (PA0)
- net at X1.3 (OUT): now also U4.5 (PF0)
Other:
- moved on the sheet: D7, Q1, Q3, Q4, Q5, R16, R17, R18, U6

Commit message: feat: enable dac
Connections:
- net ROT_A: now also U4.15 (PA7); no longer U4.10 (PA2)
- net ROT_B: now also U4.16 (PB0); no longer U4.11 (PA3)
- net ROT_SW: now also U4.14 (PA6); no longer U4.9 (PA1)
- net SLEEP: now reaches D1.3 (COM), R1.2
- net SLEEP: now also U4.13 (PA5); no longer U4.8 (PA0)
- net ADC2_IN3 renamed ADC1_IN3
- net ADC1_IN3: now also U4.10 (PA2); no longer U4.14 (PA6)
- net TEMP_210 renamed ADC2_IN2
- net ADC2_IN2: now also U4.9 (PA1)
- net TEMP_245 renamed ADC2_IN1
- net ADC2_IN1: now also U4.8 (PA0)
Other:
- moved on the sheet: D1, R1, TP1

Commit message: fix: adc assignments
Connections:
- net CURR_OUT is gone; now on net ADC1_IN4: C32.1, R29.1
- net CURR_ALERT: no longer U4.22 (PB10)
- net ADC1_IN4: now reaches U4.11 (PA3)
Other:
- moved on the sheet: C30, R30
Changed lines of the file:
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@@
 	(wire
 		(pts
-			(xy 367.03 219.71) (xy 367.03 220.98)
+			(xy 355.6 231.14) (xy 355.6 232.41)
 		)
 		(stroke
@@
 	(wire
 		(pts
-			(xy 393.7 229.87) (xy 393.7 232.41)
+			(xy 382.27 241.3) (xy 382.27 243.84)
 		)
 		(stroke
@@
 	(wire
 		(pts
-			(xy 393.7 219.71) (xy 393.7 222.25)
+			(xy 382.27 231.14) (xy 382.27 233.68)
 		)
 		(stroke
@@
 	(wire
 		(pts
-			(xy 382.27 234.95) (xy 367.03 234.95)
+			(xy 370.84 246.38) (xy 355.6 246.38)
 		)
 		(stroke
@@
 	(wire
 		(pts
-			(xy 166.37 82.55) (xy 182.88 82.55)
-		)
-		(stroke
-			(width 0)
-			(type default)
-		)
-	)
-	(wire
-		(pts
 			(xy 312.42 68.58) (xy 312.42 69.85)
 		)
@@
 	(wire
 		(pts
+			(xy 215.9 36.83) (xy 232.41 36.83)
+		)
+		(stroke
+			(width 0)
+			(type default)
+		)
+	)
+	(wire
+		(pts
 			(xy 127 69.85) (xy 127 72.39)
 		)
@@
 	(wire
 		(pts
-			(xy 355.6 223.52) (xy 344.17 223.52)
+			(xy 344.17 223.52) (xy 372.11 223.52)
 		)
 		(stroke
@@
 	(wire
 		(pts
-			(xy 367.03 228.6) (xy 367.03 234.95)
+			(xy 355.6 240.03) (xy 355.6 246.38)
 		)
 		(stroke
@@
 		)
 	)
+	(label "ADC1_IN4"
+		(at 232.41 36.83 180)
+		(fields_autoplaced yes)
+		(effects
+			(font
+				(size 1.524 1.524)
+			)
+			(justify right bottom)
+		)
+	)
 	(label "VOLTAGE"
 		(at 52.07 104.14 180)
@@
 		)
 	)
+	(label "ADC1_IN4"
+		(at 372.11 223.52 180)
+		(fields_autoplaced yes)
+		(effects
+			(font
+				(size 1.524 1.524)
+			)
+			(justify right bottom)
+		)
+	)
 	(label "CURR_ALERT"
 		(at 264.16 180.34 0)
@@
 	)
 	(label "CURR_OUT"
-		(at 355.6 223.52 180)
+		(at 358.14 223.52 180)
 		(fields_autoplaced yes)
 		(effects
@@
 	)
 	(label "CURR_ALERT"
-		(at 382.27 234.95 180)
+		(at 370.84 246.38 180)
 		(fields_autoplaced yes)
 		(effects
@@
 		)
 	)
-	(label "CURR_ALERT"
-		(at 166.37 82.55 0)
-		(fields_autoplaced yes)
-		(effects
-			(font
-				(size 1.524 1.524)
-			)
-			(justify left bottom)
-		)
-	)
 	(label "OLED_D_C"
 		(at 232.41 54.61 180)
@@
 	(symbol
 		(lib_id "Device:C")
-		(at 393.7 226.06 0)
+		(at 382.27 237.49 0)
 		(mirror y)
 		(unit 1)
@@
 		(dnp no)
 		(property "Reference" "C30"
-			(at 390.779 224.8916 0)
+			(at 379.349 236.3216 0)
 			(effects
 				(font
@@
 		)
 		(property "Value" "100n"
-			(at 390.779 227.203 0)
+			(at 379.349 238.633 0)
 			(effects
 				(font
@@
 		)
 		(property "Footprint" "Capacitor_SMD:C_0603_1608Metric"
-			(at 392.7348 229.87 0)
+			(at 381.3048 241.3 0)
 			(effects
 				(font
@@
 		)
 		(property "Datasheet" "~"
-			(at 393.7 226.06 0)
+			(at 382.27 237.49 0)
 			(effects
 				(font
@@
 		)
 		(property "Description" "Unpolarized capacitor"
-			(at 393.7 226.06 0)
+			(at 382.27 237.49 0)
 			(effects
 				(font
@@
 	(symbol
 		(lib_id "Device:R")
-		(at 367.03 224.79 0)
+		(at 355.6 236.22 0)
 		(mirror x)
 		(unit 1)
@@
 		(dnp no)
 		(property "Reference" "R30"
-			(at 368.7826 225.9584 0)
+			(at 357.3526 237.3884 0)
 			(effects
 				(font
@@
 		)
 		(property "Value" "10k"
-			(at 368.7826 223.647 0)
+			(at 357.3526 235.077 0)
 			(effects
 				(font
@@
 		)
 		(property "Footprint" "Resistor_SMD:R_0603_1608Metric"
-			(at 365.252 224.79 90)
+			(at 353.822 236.22 90)
 			(effects
 				(font
@@
 		)
 		(property "Datasheet" "~"
-			(at 367.03 224.79 0)
+			(at 355.6 236.22 0)
 			(effects
 				(font
@@
 		)
 		(property "Description" "Resistor"
-			(at 367.03 224.79 0)
+			(at 355.6 236.22 0)
 			(effects
 				(font
@@
 	(symbol
 		(lib_id "power:+3V3")
-		(at 367.03 219.71 0)
+		(at 355.6 231.14 0)
 		(mirror y)
 		(unit 1)
@@
 		(dnp no)
 		(property "Reference" "#PWR082"
-			(at 367.03 223.52 0)
+			(at 355.6 234.95 0)
 			(effects
 				(font
@@
 		)
 		(property "Value" "+3V3"
-			(at 366.649 215.3158 0)
+			(at 355.219 226.7458 0)
 			(effects
 				(font
@@
 		)
 		(property "Footprint" ""
-			(at 367.03 219.71 0)
+			(at 355.6 231.14 0)
 			(effects
 				(font
@@
 		)
 		(property "Datasheet" ""
-			(at 367.03 219.71 0)
+			(at 355.6 231.14 0)
 			(effects
 				(font
@@
 		)
 		(property "Description" "Power symbol creates a global label with name \"+3V3\""
-			(at 367.03 219.71 0)
+			(at 355.6 231.14 0)
 			(effects
 				(font
@@
 	(symbol
 		(lib_id "power:GND")
-		(at 393.7 232.41 0)
+		(at 382.27 243.84 0)
 		(mirror y)
 		(unit 1)
@@
 		(dnp no)
 		(property "Reference" "#PWR085"
-			(at 393.7 238.76 0)
+			(at 382.27 250.19 0)
 			(effects
 				(font
@@
 		)
 		(property "Value" "GND"
-			(at 393.573 236.8042 0)
+			(at 382.143 248.2342 0)
 			(effects
 				(font
@@
 		)
 		(property "Footprint" ""
-			(at 393.7 232.41 0)
+			(at 382.27 243.84 0)
 			(effects
 				(font
@@
 		)
 		(property "Datasheet" ""
-			(at 393.7 232.41 0)
+			(at 382.27 243.84 0)
 			(effects
 				(font
@@
 		)
 		(property "Description" "Power symbol creates a global label with name \"GND\" , ground"
-			(at 393.7 232.41 0)
+			(at 382.27 243.84 0)
 			(effects
 				(font
@@
 	(symbol
 		(lib_id "power:+3V3")
-		(at 393.7 219.71 0)
+		(at 382.27 231.14 0)
 		(mirror y)
 		(unit 1)
@@
 		(dnp no)
 		(property "Reference" "#PWR083"
-			(at 393.7 223.52 0)
+			(at 382.27 234.95 0)
 			(effects
 				(font
@@
 		)
 		(property "Value" "+3V3"
-			(at 393.319 215.3158 0)
+			(at 381.889 226.7458 0)
 			(effects
 				(font
@@
 		)
 		(property "Footprint" ""
-			(at 393.7 219.71 0)
+			(at 382.27 231.14 0)
 			(effects
 				(font
@@
 		)
 		(property "Datasheet" ""
-			(at 393.7 219.71 0)
+			(at 382.27 231.14 0)
 			(effects
 				(font
@@
 		)
 		(property "Description" "Power symbol creates a global label with name \"+3V3\""
-			(at 393.7 219.71 0)
+			(at 382.27 231.14 0)
 			(effects
 				(font

Commit message: feat: add further pins
Connections:
- net CURR_ALERT: now also U4.4 (PC15)
- net ROT_A: now also U4.17 (PB1); no longer U4.15 (PA7)
- net ROT_B: now also U4.18 (PB2); no longer U4.16 (PB0)
- net ROT_SW: now also U4.16 (PB0); no longer U4.14 (PA6)
Changed lines of the file:
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@@
 	(wire
 		(pts
-			(xy 215.9 46.99) (xy 232.41 46.99)
-		)
-		(stroke
-			(width 0)
-			(type default)
-		)
-	)
-	(wire
-		(pts
 			(xy 330.2 133.35) (xy 334.01 133.35)
 		)
@@
 	(wire
 		(pts
-			(xy 182.88 57.15) (xy 166.37 57.15)
-		)
-		(stroke
-			(width 0)
-			(type default)
-		)
-	)
-	(wire
-		(pts
 			(xy 153.67 114.3) (xy 153.67 113.03)
 		)
@@
 	(wire
 		(pts
+			(xy 166.37 52.07) (xy 182.88 52.07)
+		)
+		(stroke
+			(width 0)
+			(type default)
+		)
+	)
+	(wire
+		(pts
 			(xy 53.34 71.12) (xy 53.34 72.39)
 		)
@@
 	(wire
 		(pts
+			(xy 182.88 57.15) (xy 166.37 57.15)
+		)
+		(stroke
+			(width 0)
+			(type default)
+		)
+	)
+	(wire
+		(pts
 			(xy 374.65 71.12) (xy 374.65 72.39)
 		)
@@
 		)
 	)
-	(wire
-		(pts
-			(xy 215.9 44.45) (xy 232.41 44.45)
-		)
-		(stroke
-			(width 0)
-			(type default)
-		)
-	)
 	(polyline
 		(pts
@@
 	(wire
 		(pts
+			(xy 182.88 62.23) (xy 166.37 62.23)
+		)
+		(stroke
+			(width 0)
+			(type default)
+		)
+	)
+	(wire
+		(pts
 			(xy 284.48 215.9) (xy 284.48 219.71)
 		)
@@
 	(wire
 		(pts
+			(xy 182.88 59.69) (xy 166.37 59.69)
+		)
+		(stroke
+			(width 0)
+			(type default)
+		)
+	)
+	(wire
+		(pts
 			(xy 132.08 35.56) (xy 140.97 35.56)
 		)
@@
 		)
 	)
+	(label "ROT_A"
+		(at 166.37 59.69 0)
+		(fields_autoplaced yes)
+		(effects
+			(font
+				(size 1.524 1.524)
+			)
+			(justify left bottom)
+		)
+	)
 	(label "SHUNT-"
 		(at 374.65 160.02 180)
@@
 		)
 	)
+	(label "ROT_SW"
+		(at 166.37 57.15 0)
+		(fields_autoplaced yes)
+		(effects
+			(font
+				(size 1.524 1.524)
+			)
+			(justify left bottom)
+		)
+	)
 	(label "CC2"
 		(at 55.88 36.83 180)
@@
 		)
 	)
-	(label "ROT_A"
-		(at 232.41 46.99 180)
-		(fields_autoplaced yes)
-		(effects
-			(font
-				(size 1.524 1.524)
-			)
-			(justify right bottom)
-		)
-	)
 	(label "NRST"
 		(at 130.81 72.39 0)
@@
 		)
 	)
-	(label "ROT_B"
-		(at 166.37 57.15 0)
-		(fields_autoplaced yes)
-		(effects
-			(font
-				(size 1.524 1.524)
-			)
-			(justify left bottom)
-		)
-	)
 	(label "SWO"
 		(at 166.37 64.77 0)
@@
 		)
 	)
-	(label "ROT_SW"
-		(at 232.41 44.45 180)
+	(label "ROT_B"
+		(at 166.37 62.23 0)
 		(fields_autoplaced yes)
 		(effects
@@
 				(size 1.524 1.524)
 			)
-			(justify right bottom)
+			(justify left bottom)
 		)
 	)
@@
 		(fields_autoplaced yes)
 		(effects
+			(font
+				(size 1.524 1.524)
+			)
+			(justify left bottom)
+		)
+	)
+	(label "CURR_ALERT"
+		(at 166.37 52.07 0)
+		(fields_autoplaced yes)
+		(effects

Commit message: feat: rev a production version
Parts:
- removed C16: 100n, Capacitor_SMD:C_0603_1608Metric, symbol Device:C
- removed C26, C31: DNP, Capacitor_SMD:C_0603_1608Metric, symbol Device:C
- removed C27: 330p, Capacitor_SMD:C_0603_1608Metric, symbol Device:C
- removed D3: BZX84Cxx, Package_TO_SOT_SMD:TSOT-23_HandSoldering, symbol custom:BZX84Cxx
- removed D8: BAT54S, Package_TO_SOT_SMD:SOT-23, symbol Diode:BAT54S
- removed J3: AudioJack3, custom:CUI_SJ-3502-SMT, symbol Connector:AudioJack3
- removed Q2: FDS6630A, Package_SO:SOIC-8_3.9x4.9mm_P1.27mm, symbol Transistor_FET:FDS6630A
- removed R21, R27: 10k, Resistor_SMD:R_0603_1608Metric, symbol Device:R
- removed R31: 220k, Resistor_SMD:R_0603_1608Metric, symbol Device:R
- removed R33: 1k, Resistor_SMD:R_0603_1608Metric, symbol Device:R
- removed U7: Opamp_Dual, Package_SO:VSSOP-8_3x3mm_P0.65mm, symbol Device:Opamp_Dual
- added C22, C23, C33: 1u, Capacitor_SMD:C_0603_1608Metric, symbol Device:C
- added C32: 100n, Capacitor_SMD:C_0603_1608Metric, symbol Device:C
- added D4: BAT54S, Package_TO_SOT_SMD:SOT-23, symbol Diode:BAT54S
- added FB1: 600@100MHz, Inductor_SMD:L_0603_1608Metric, symbol Device:FerriteBead
- added Q1: Si4162DY, Package_SO:SOIC-8_3.9x4.9mm_P1.27mm, symbol Transistor_FET:Si4162DY
- added R11: 10k, Resistor_SMD:R_0603_1608Metric, symbol Device:R
- added R20: 220k, Resistor_SMD:R_0603_1608Metric, symbol Device:R
- added R22: 33k, Resistor_SMD:R_0603_1608Metric, symbol Device:R
- added SW3: RESET, Button_Switch_SMD:SW_SPST_TL3342, symbol Switch:SW_SPST
- added TP2: 2P, Connector_Wire:SolderWire-0.75sqmm_1x01_D1.25mm_OD2.3mm, symbol Connector:TestPoint
- added TP3: 3T, Connector_Wire:SolderWire-0.75sqmm_1x01_D1.25mm_OD2.3mm, symbol Connector:TestPoint
- added TP4: 4D, Connector_Wire:SolderWire-0.75sqmm_1x01_D1.25mm_OD2.3mm, symbol Connector:TestPoint
- added TP5: 5S, Connector_Wire:SolderWire-0.75sqmm_1x01_D1.25mm_OD2.3mm, symbol Connector:TestPoint
- added U8: TLV333-DBV, Package_TO_SOT_SMD:SOT-23-5, symbol custom:TLV333-DBV
- added oshw1: Logo_Open_Hardware_Large, Symbol:OSHW-Symbol_6.7x6mm_SilkScreen, symbol Graphic:Logo_Open_Hardware_Large
- C1, C14, C15, C17, C18, C4, C5: MPN C307331 -> C14663
- C11, C12: value 1u -> 330p; MPN C15849 -> C1664
- C13: renamed from C24; MPN C307331 -> C14663
- C19: renamed from C21; MPN C307331 -> C14663
- C20: renamed from C22; MPN C307331 -> C14663
- C21: renamed from C23; MPN C307331 -> C14663
- C24: renamed from C13; footprint Capacitor_THT:C_Radial_D10.0mm_H12.5mm_P5.00mm -> Capacitor_THT:CP_Radial_D10.0mm_P3.50mm; symbol Device:CP -> Device:C_Polarized
- C25: value DNP -> 100n; MPN (none) -> C14663
- C28: value 330p -> 10u; footprint Capacitor_SMD:C_0603_1608Metric -> Capacitor_SMD:C_1206_3216Metric; MPN (none) -> C13585
- C29: value DNP -> 330p; MPN (none) -> C1664
- C30: renamed from C32; MPN (none) -> C14663
- C31: renamed from C30; MPN (none) -> C14663
- C6: MPN C307331 -> C14663; now not fitted
- D1: renamed from D4; MPN (none) -> C1974707
- D2: renamed from D6; MPN (none) -> C83935
- D3: renamed from D1; MPN (none) -> C83935
- D5: renamed from D2; MPN (none) -> C83935
- D6: renamed from D7; MPN (none) -> C8598
- D7: renamed from D5; MPN (none) -> C83935
- J2: value USB_C_Receptacle_USB2.0 -> USB_C_Receptacle_USB2.0_16P; footprint Connector_USB:USB_C_Receptacle_G-Switch_GT-USB-7010ASV -> Connector_USB:USB_C_Receptacle_HRO_TYPE-C-31-M-12; symbol Connector:USB_C_Receptacle_USB2.0 -> Connector:USB_C_Receptacle_USB2.0_16P; MPN C2988369 -> C165948
- Q2: renamed from Q1; MPN (none) -> C466643
- Q3: MPN (none) -> C3289788
- Q4: MPN (none) -> C466643
- Q5: MPN (none) -> C466642
- R1: renamed from R2; MPN C25105 -> C23140
- R10: renamed from R1; MPN (none) -> C25804
- R12: renamed from R23; MPN (none) -> C25804
- R13: renamed from R24; value TBD -> 620
- R14: renamed from R10; MPN (none) -> C25804
- R15: renamed from R11; MPN (none) -> C25804
- R16: renamed from R12; MPN (none) -> C25804
- R17: renamed from R13; MPN (none) -> C25804
- R18: renamed from R14; MPN (none) -> C25804
- R19: renamed from R15; MPN (none) -> C25804
- R2: renamed from R3; MPN C25105 -> C23140
- R21: renamed from R16; MPN (none) -> C21190
- R23: renamed from R17; value 0.47 -> 1; MPN (none) -> C22936
- R24: renamed from R18; MPN (none) -> C21190
- R25: renamed from R19; MPN (none) -> C22935
- R26: value 1M -> 10k; MPN (none) -> C25804
- R27: renamed from R22; MPN (none) -> C22961
- R28: renamed from R25; MPN (none) -> C21190
- R29: renamed from R28; MPN (none) -> C844087
- R3: renamed from R4; value 5.1k -> 10k; MPN C25905 -> C25804
- R30: renamed from R29; MPN (none) -> C25804
- R32: renamed from R30; MPN (none) -> C25804
- R4: renamed from R5; value 5.1k -> 10k; MPN C25905 -> C25804
- R5: renamed from R6; value 5.1k -> 10k; MPN C25905 -> C25804
- R6: renamed from R7; value 5.1k -> 10k; MPN C25905 -> C25804
- R7: renamed from R20; MPN (none) -> C25804
- R8: MPN (none) -> C25804
- R9: value 1k -> 10k; MPN (none) -> C25804
- TP1: value SLEEP -> 1C; footprint TestPoint:TestPoint_THTPad_D2.0mm_Drill1.0mm -> Connector_Wire:SolderWire-0.75sqmm_1x01_D1.25mm_OD2.3mm
- U1: MPN (none) -> C7519
- U4: MPN (none) -> C529355
- U5: renamed from U8; value ~ -> TCPP01-M12
- U6: MPN (none) -> C459531
- U9: value INA301 -> INA301A1
- X1: now not fitted
- renumbered C19 to C26, C20 to C27, R32 to R31, U5 to U7
Connections:
- net +3V3: now also C28.1, R12.1, R8.1, R9.1, U5.10 (~{DB}), D4.2 (K), FB1.1, U8.5 (V+); no longer R12.2, R26.1, U4.21 (VDDA)
- net ADC1_IN3: now also R20.2, R22.2; no longer R8.1, R9.2
- net ADC2_IN1: now also C29.1, R27.1, U8.1
- net ADC2_IN2: now also D4.3 (COM), R11.2; no longer R27.1
- net CC1: now also C12.1
- net CC2: now also C11.1
- net CURR_ALERT: now also U4.25 (PB11); no longer U4.4 (PC15)
- net GND: now also TP1.1, U9.5 (RESET), C22.1, C23.1, C32.2, C33.1, D4.1 (A), R22.1, SW3.1 (A), U8.2 (V-); no longer C29.2, R9.1
- net NRST: now also SW3.2 (B)
- net SLEEP: now also R10.1, R8.2, TP5.1; no longer D3.3 (COM), R10.2, U4.13 (PA5)
- net UCPD_CC1: no longer C28.1
- net VBUS: now also C22.2, C23.2, Q1.5 (D), Q1.6 (D), Q1.7 (D), Q1.8 (D); no longer C11.1, C12.1
- net VDC: now also Q1.1 (S), Q1.2 (S), Q1.3 (S), R20.1; no longer R8.2
- net at R27.2, R28.1: now also C29.2, U8.4 (-)
- net at D7.3 (COM): now also C25.1, R26.2, U8.3 (+)
- net at U5.11 (~{FLT}): now also R12.2; no longer R12.1
- net at U5.5 (GATE): now also Q1.4 (G)
- net _SLEEP: now reaches U4.22 (PB10)
- net _SLEEP: now also D3.3 (COM), R10.2
- net CURR_RESET renamed TIM1_CH1
- net TIM1_CH1: now also U6.1; no longer U9.5 (RESET)
- removed net DETECT/210: C29.1, R26.2
- net HEATER/245 renamed HEATER
- net HEATER: now also TP2.1; no longer C25.1, R25.2
- removed net TIM2_CH4: U4.25 (PB11), U6.1
- new net DET: R11.1, R9.2, TP4.1
- new net TC+: R25.2, R26.1, TP3.1
- new net VDDA: C32.1, C33.2, FB1.2, U4.21 (VDDA)
- no-connect marks 4 -> 13
Other:
- note added: "22 V limit"
- note added: ">20 V Vds specified at 5 V Vgs"
- note added: ">20 V Vgs, >20 V Vds minimum requirement for PMOS"
- note added: "C210 1_COM: green+blue 2_TC+: red 3_HEATER: red"
- note added: "C245 1_COM: green 2_TC+: red 3_HEATER: blue"
- note added: "Feedback: 2180 Hz low-pass"
- note added: "Input: 160 Hz low-pass"
- note added: "RESET low: Transparent alert mode"
- note added: "Thermocouple amplifier"
- note added: "VOGT 1018.68"
- note removed: "20 V Vgs, 20 V Vds minimum requirement for PMOS"
- note removed: "C210 Sleeve: green (COM/GND) Ring: blue (detect) Tip: red (TC+/series HEATER)"
- note removed: "C245 Sleeve: green (COM/GND) Ring: red (TC+) Tip: blue (HEATER)"
- note removed: "Thermocouple amplifiers"
- company: (none) -> elagil
- title: (none) -> loeti
- moved on the sheet: C13, C17, C18, C24, C26, C27, C30, C31, D1, D2, D3, D5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

Commit message: feat: full features
Parts:
- removed C6: 100n, Capacitor_SMD:C_0603_1608Metric, symbol Device:C
- removed R1, R2: 33, Resistor_SMD:R_0603_1608Metric, symbol Device:R
- removed SW3: RESET, Button_Switch_SMD:SW_SPST_TL3342, symbol Switch:SW_SPST
- removed U1: USBLC6-2SC6, Package_TO_SOT_SMD:SOT-23-6, symbol Power_Protection:USBLC6-2SC6
- removed U7: AMS1117-3.3, Package_TO_SOT_SMD:SOT-223-3_TabPin2, symbol Regulator_Linear:AMS1117-3.3
- removed X1: SG-210STF (16 MHz), Oscillator:Oscillator_SMD_SeikoEpson_SG210-4Pin_2.5x2.0mm, symbol Oscillator:SG-210STF
- added C28: 1u, Capacitor_SMD:C_0603_1608Metric, symbol Device:C
- added C31: 10u, Capacitor_SMD:C_1206_3216Metric, symbol Device:C
- added J3: USB_C_Receptacle_USB2.0_16P, Connector_USB:USB_C_Receptacle_HRO_TYPE-C-31-M-12, symbol Connector:USB_C_Receptacle_USB2.0_16P
- added L1: 10u, Inductor_SMD:L_Abracon_ASPI-0425, symbol Device:L
- added R33, R34: 33, Resistor_SMD:R_0603_1608Metric, symbol Device:R
- added U10: TPS62177DQC, Package_SON:WSON-10-1EP_2x3mm_P0.5mm_EP0.84x2.4mm_ThermalVias, symbol Regulator_Switching:TPS62177DQC
- added U7: USBLC6-2SC6, Package_TO_SOT_SMD:SOT-23-6, symbol Power_Protection:USBLC6-2SC6
- C25: renamed from C24; value 68u -> 82u
- C27: value 10u -> 100n; footprint Capacitor_SMD:C_1206_3216Metric -> Capacitor_SMD:C_0603_1608Metric; MPN C13585 -> C14663
- TP2: value 2P -> 3P
- TP3: value 3T -> 2T
- renumbered C8 to C10, C9 to C11, C10 to C12, C11 to C13, C12 to C14, C13 to C15, C14 to C16, C15 to C17, C17 to C18, C18 to C19, C33 to C2, C19 to C20, C20 to C21, C21 to C22, C22 to C23, C23 to C24, C32 to C3, C28 to C30, C29 to C32, C25 to C33, C30 to C34, C31 to C35, C2 to C4, C3 to C5, C4 to C6, C5 to C7, C7 to C9, SW2 to SW3
Connections:
- net +3V3: now also C31.1, L1.2, U10.10 (VOS), U10.8 (~{SLEEP}); no longer U5.10 (~{DB})
- net GND: now also C27.1, C28.1, C31.2, J3.A1 (GND), J3.A12 (GND), J3.B1 (GND), J3.B12 (GND), J3.S1 (SHIELD), U10.1 (PGND), U10.11 (PAD), U10.4 (NC), U10.5 (FB), U10.6 (AGND), U7.2 (GND); no longer C27.2
- net USB_D_N: now also R33.2
- net USB_D_P: now also R34.2
- net VDC: now also U10.2 (VIN), U10.3 (EN); no longer C27.1
- net _USB_D_N: now also R33.1, U7.6 (I/O1)
- net _USB_D_P: now also R34.1, U7.4 (I/O2)
- net at J2.A7 (D-): no longer J2.B7 (D-)
- net at J2.A6 (D+): no longer J2.B6 (D+)
- net VREF+: now reaches U4.20 (VREF+)
- net VREF+: now also C27.2, C28.2
- net UCPD_DB: now reaches U4.42 (PB5)
- net UCPD_DB: now also U5.10 (~{DB})
- new net: L1.1, U10.9 (SW)
- new net: J3.A7 (D-), J3.B7 (D-), U7.1 (I/O1)
- new net: J3.A6 (D+), J3.B6 (D+), U7.3 (I/O2)
- new net: J3.A4 (VBUS), J3.A9 (VBUS), J3.B4 (VBUS), J3.B9 (VBUS), U7.5 (VBUS)
- no-connect marks 13 -> 21
Other:
- title: loeti -> loeti v6
- moved on the sheet: C13, C14, C15, C23, C24, C25, C26, C30, D1, D2, D5, J2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

Commit message: chore: clean up submodules
Parts:
- added C29, C8: 10u, Capacitor_SMD:C_1206_3216Metric, symbol Device:C
- added D8, D9: B5819W SL, Diode_SMD:D_SOD-123, symbol Device:D_Schottky
- added L2: 10u, Inductor_SMD:L_Abracon_ASPI-0630LR, symbol Device:L
- C33: value 100n -> DNP
- J2: value USB_C_Receptacle_USB2.0_16P -> POWER
- J3: value USB_C_Receptacle_USB2.0_16P -> DEBUG
Connections:
- net GND: now also C29.2, C8.2
- net HEATER: now also C29.1, C8.1, L2.2; no longer D6.1 (K), Q3.5 (D), Q3.6 (D), Q3.7 (D), Q3.8 (D)
- net VDC: now also D9.2 (A); no longer U10.2 (VIN), U10.3 (EN)
- net +5VP: now reaches J3.A4 (VBUS), J3.A9 (VBUS), J3.B4 (VBUS), J3.B9 (VBUS), U7.5 (VBUS)
- net +5VP: now also D8.2 (A)
- new net: D6.1 (K), L2.1, Q3.5 (D), Q3.6 (D), Q3.7 (D), Q3.8 (D)
- new net: D8.1 (K), D9.1 (K), U10.2 (VIN), U10.3 (EN)
Other:
- note added: "159.2 Hz low-pass Settles to 0.01 % in 9.2 ms"
- note removed: "159.2 Hz low-pass"
- note removed: "Input: 160 Hz low-pass"
- moved on the sheet: C13, C14, C15, C23, C24, C25, C26, C30, C31, D1, D2, D5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

Commit message: fix: working revision
Parts:
- removed C29, C8: 10u, Capacitor_SMD:C_1206_3216Metric, symbol Device:C
- removed L2: 10u, Inductor_SMD:L_Abracon_ASPI-0630LR, symbol Device:L
Connections:
- net HEATER: now also D6.1 (K), Q3.5 (D), Q3.6 (D), Q3.7 (D), Q3.8 (D)
