File: hardware/loeti.kicad_pcb (KiCad board)
At the start: 4 copper layers, 80 x 50.5 mm, 94 parts, among them J1 REDFIT_SWD_6, J2 USB_C_Receptacle_USB2.0, J3 AudioJack3, Q1 BC817, Q2 FDS6630A, Q3 Si4425FDY, Q4 BC817, Q5 BC807, SW1 BOOT, SW2 RotaryEncoder_Switch, U1 USBLC6-2SC6, U2 EA_OLEDS102-6, U3 M24C64-RMN, U4 STM32G431CBTx, U5 AMS1117-3.3, U6 74AHC1G08, U7 Opamp_Dual, U9 INA301, X1 SG-210STF (16 MHz)

Commit message: feat: rev a production version
Parts:
- removed C16: 100n, Capacitor_SMD:C_0603_1608Metric
- removed the C26 at (127.4, 108.1)
- removed the C27 at (132.8, 83.6)
- removed the C30 at (126.5, 105.0)
- removed the D3 at (143.1, 105.5)
- removed the D5 at (123.6, 104.7)
- removed D8: BAT54S, Package_TO_SOT_SMD:SOT-23
- removed J3: AudioJack3, custom:CUI_SJ-3502-SMT
- removed the Q2 at (124.6, 89.4)
- removed the R19 at (120.0, 103.5)
- removed the R21 at (119.5, 105.1)
- removed the R31 at (125.8, 111.6)
- removed R33: 1k, Resistor_SMD:R_0603_1608Metric
- removed the U7 at (123.0, 109.9)
- added C22: 1u, Capacitor_SMD:C_0603_1608Metric, F.Cu at (120.2, 107.9)
- added C23: 1u, Capacitor_SMD:C_0603_1608Metric, F.Cu at (118.6, 107.9)
- added C32: 100n, Capacitor_SMD:C_0603_1608Metric, F.Cu at (153.1, 83.5)
- added C33: 1u, Capacitor_SMD:C_0603_1608Metric, F.Cu at (151.4, 83.5)
- added D4: BAT54S, Package_TO_SOT_SMD:SOT-23, F.Cu at (124.5, 85.1)
- added D7: BAT54S, Package_TO_SOT_SMD:SOT-23, F.Cu at (135.2, 86.6)
- added FB1: 600@100MHz, Inductor_SMD:L_0603_1608Metric, F.Cu at (149.8, 83.5)
- added Q1: Si4162DY, Package_SO:SOIC-8_3.9x4.9mm_P1.27mm, F.Cu at (125.0, 112.8)
- added R11: 10k, Resistor_SMD:R_0603_1608Metric, F.Cu at (123.8, 81.5)
- added R20: 220k, Resistor_SMD:R_0603_1608Metric, F.Cu at (140.3, 96.0)
- added R28: 1k, Resistor_SMD:R_0603_1608Metric, F.Cu at (133.1, 77.0)
- added SW3: RESET, Button_Switch_SMD:SW_SPST_TL3342, F.Cu at (176.2, 97.6)
- added TP2: 2P, Connector_Wire:SolderWire-0.75sqmm_1x01_D1.25mm_OD2.3mm, F.Cu at (108.9, 94.0)
- added TP3: 3T, Connector_Wire:SolderWire-0.75sqmm_1x01_D1.25mm_OD2.3mm, F.Cu at (124.0, 88.9)
- added TP4: 4D, Connector_Wire:SolderWire-0.75sqmm_1x01_D1.25mm_OD2.3mm, F.Cu at (124.0, 78.1)
- added TP5: 5S, Connector_Wire:SolderWire-0.75sqmm_1x01_D1.25mm_OD2.3mm, F.Cu at (127.9, 78.1)
- added U8: TLV333-DBV, Package_TO_SOT_SMD:SOT-23-5, F.Cu at (133.8, 83.0)
- added oshw1: Logo_Open_Hardware_Large, Symbol:OSHW-Symbol_6.7x6mm_SilkScreen, F.Cu at (182.8, 104.1)
- C11, C12: value 1u -> 330p
- C24: renamed from C13; footprint Capacitor_THT:C_Radial_D10.0mm_H12.5mm_P5.00mm -> Capacitor_THT:CP_Radial_D10.0mm_P3.50mm
- C25, C31: value DNP -> 100n
- C28: value 330p -> 10u; footprint Capacitor_SMD:C_0603_1608Metric -> Capacitor_SMD:C_1206_3216Metric
- C29: value DNP -> 330p
- J2: value USB_C_Receptacle_USB2.0 -> USB_C_Receptacle_USB2.0_16P; footprint Connector_USB:USB_C_Receptacle_G-Switch_GT-USB-7010ASV -> Connector_USB:USB_C_Receptacle_HRO_TYPE-C-31-M-12
- R13: renamed from R24; value TBD -> 620
- R22: value 220k -> 33k
- R23: renamed from R17; value 0.47 -> 1
- R25: value 1k -> 1M
- R26: value 1M -> 10k
- R27: value 10k -> 220k
- R3: renamed from R4; value 5.1k -> 10k
- R4: renamed from R5; value 5.1k -> 10k
- R5: renamed from R6; value 5.1k -> 10k
- R6: renamed from R7; value 5.1k -> 10k
- R9: value 1k -> 10k
- TP1: value SLEEP -> 1C; footprint TestPoint:TestPoint_THTPad_D2.0mm_Drill1.0mm -> Connector_Wire:SolderWire-0.75sqmm_1x01_D1.25mm_OD2.3mm
- U5: renamed from U8; value ~ -> TCPP01-M12
- U9: value INA301 -> INA301A1
- moved TP1 70.9 mm to (112.9, 94.0)
- moved D3 55.8 mm to (128.2, 85.1)
- moved R10 54.4 mm to (127.4, 81.5), turned to -90 degrees
- moved C29 42.1 mm to (133.1, 80.2), turned to 0 degrees
- moved R27 38.7 mm to (133.1, 78.6), turned to 0 degrees
- moved C12 38.1 mm to (131.9, 114.4), turned to -90 degrees
- moved C11 35.8 mm to (137.0, 112.0)
- moved R7 34.7 mm to (129.4, 114.6)
- moved R13 34.1 mm to (129.4, 113.0), turned to 0 degrees
- moved D2 32.3 mm to (117.8, 115.5), turned to 0 degrees
- moved R26 31.7 mm to (131.6, 87.2), turned to 0 degrees
- moved C13 31.4 mm to (134.2, 113.6), turned to 180 degrees
- moved C28 29.5 mm to (146.5, 108.1), turned to 90 degrees
- moved D1 29.0 mm to (117.0, 107.9)
- moved U1 28.5 mm to (117.5, 111.2)
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- renumbered C24 to C13, C21 to C19, C22 to C20, C23 to C21, C19 to C26, C20 to C27, C32 to C30, D4 to D1, D6 to D2, D1 to D3, D2 to D5, D7 to D6, Q1 to Q2, R2 to R1, R1 to R10, R23 to R12, R10 to R14, R11 to R15, R12 to R16, R13 to R17, R14 to R18, R15 to R19, R3 to R2, R16 to R21, R18 to R24, R28 to R29, R29 to R30, R32 to R31, R30 to R32, R20 to R7, U5 to U7
Connections:
- C11 pad 1: VBUS -> /CC2
- C12 pad 1: VBUS -> /CC1
- C25 pad 1: /HEATER/245 -> Net-(D7-COM)
- C28 pad 1: /UCPD_CC1 -> +3V3
- C29 pad 1: /DETECT/210 -> /ADC2_IN1
- C29 pad 2: GND -> Net-(U8--)
- C31 pad 1: /ADC2_IN1 -> +3V3
- C31 pad 2: Net-(U7B--) -> GND
- D3 pad 3: /SLEEP -> /_SLEEP
- D6 pad 1: /HEATER/245 -> /HEATER
- Q3 pad 5: /HEATER/245 -> /HEATER
- Q3 pad 6: /HEATER/245 -> /HEATER
- Q3 pad 7: /HEATER/245 -> /HEATER
- Q3 pad 8: /HEATER/245 -> /HEATER
- R10 pad 1: Net-(R1-Pad1) -> /SLEEP
- R10 pad 2: /SLEEP -> /_SLEEP
- R12 pad 1: Net-(U8-~{FLT}) -> +3V3
- R12 pad 2: +3V3 -> Net-(U5-~{FLT})
- R22 pad 1: /ADC2_IN2 -> GND
- R22 pad 2: Net-(U7A--) -> /ADC1_IN3
- R25 pad 1: Net-(U7A--) -> +3V3
- R25 pad 2: GND -> /TC+
- R26 pad 1: +3V3 -> /TC+
- R26 pad 2: /DETECT/210 -> Net-(D7-COM)
- R27 pad 1: Net-(D8-COM) -> /ADC2_IN1
- R27 pad 2: /DETECT/210 -> Net-(U8--)
- R8 pad 1: /ADC1_IN3 -> +3V3
- R8 pad 2: VDC -> /SLEEP
- R9 pad 1: GND -> +3V3
- R9 pad 2: /ADC1_IN3 -> /DET
- TP1 pad 1: Net-(R1-Pad1) -> GND
- U4 pad 13: /SLEEP -> unconnected-(U4-PA5-Pad13)
- U4 pad 21: +3V3 -> /VDDA
- U4 pad 22: unconnected-(U4-PB10-Pad22) -> /_SLEEP
- U4 pad 25: /TIM2_CH4 -> /CURR_ALERT
- U4 pad 30: /CURR_RESET -> /TIM1_CH1
- U4 pad 4: /CURR_ALERT -> unconnected-(U4-PC15-Pad4)
- U5 pad 10: unconnected-(U8-~{DB}-Pad10) -> +3V3
- U5 pad 11: Net-(U8-~{FLT}) -> Net-(U5-~{FLT})
- U6 pad 1: /TIM2_CH4 -> /TIM1_CH1
- U9 pad 5: /CURR_RESET -> GND
Routing:
- net /TIM2_CH4: track 40.1 -> 0.00 mm, vias 2 -> 0
- net /CURR_RESET: track 39.3 -> 0.00 mm, vias 2 -> 0
- net /_SLEEP: track 0.00 -> 30.4 mm, vias 0 -> 2
- net /SLEEP: track 28.9 -> 3.68 mm
- net /TIM1_CH1: track 0.00 -> 22.6 mm
- net /ADC2_IN1: track 55.5 -> 40.9 mm
- net Net-(D2-COM): track 4.23 -> 18.7 mm
- net /CURR_ALERT: track 52.6 -> 40.2 mm
- net /CC2: track 15.0 -> 26.3 mm
- net /HEATER/245: track 11.2 -> 0.00 mm
- net Net-(Q1-G): track 21.8 -> 10.7 mm
- net /DETECT/210: track 10.2 -> 0.00 mm
- net /CC1: track 15.1 -> 24.6 mm
- net /BOOT0: track 27.5 -> 18.1 mm
- net /ADC2_IN2: track 52.4 -> 43.6 mm
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- added copper zone on F.Cu, net /HEATER
- removed copper zone on F.Cu, net /HEATER/245
Other:
- outline, holes or cut-outs redrawn

Commit message: feat: full features
Parts:
- removed the C6 at (164.0, 93.0)
- removed R1, R2: 33, Resistor_SMD:R_0603_1608Metric
- removed the SW3 at (176.2, 97.6)
- removed U1: USBLC6-2SC6, Package_TO_SOT_SMD:SOT-23-6
- removed X1: SG-210STF (16 MHz), Oscillator:Oscillator_SMD_SeikoEpson_SG210-4Pin_2.5x2.0mm
- added C28: 1u, Capacitor_SMD:C_0603_1608Metric, F.Cu at (152.4, 83.2)
- added C31: 10u, Capacitor_SMD:C_1206_3216Metric, F.Cu at (147.5, 105.7)
- added J3: USB_C_Receptacle_USB2.0_16P, Connector_USB:USB_C_Receptacle_HRO_TYPE-C-31-M-12, F.Cu at (182.8, 92.9)
- added L1: 10u, Inductor_SMD:L_Abracon_ASPI-0425, F.Cu at (144.5, 110.5)
- added R33: 33, Resistor_SMD:R_0603_1608Metric, F.Cu at (146.8, 92.0)
- added R34: 33, Resistor_SMD:R_0603_1608Metric, F.Cu at (146.8, 93.6)
- added U10: TPS62177DQC, Package_SON:WSON-10-1EP_2x3mm_P0.5mm_EP0.84x2.4mm_ThermalVias, F.Cu at (141.8, 106.2)
- C25: renamed from C24; value 68u -> 82u
- C27: value 10u -> 100n; footprint Capacitor_SMD:C_1206_3216Metric -> Capacitor_SMD:C_0603_1608Metric
- TP2: value 2P -> 3P
- TP3: value 3T -> 2T
- U7: value AMS1117-3.3 -> USBLC6-2SC6; footprint Package_TO_SOT_SMD:SOT-223-3_TabPin2 -> Package_TO_SOT_SMD:SOT-23-6
- moved U7 35.1 mm to (174.0, 93.1), turned to 180 degrees
- moved C27 19.9 mm to (154.0, 83.2), turned to -90 degrees
- moved D5 7.94 mm to (136.9, 98.9), turned to 0 degrees
- moved oshw1 5.88 mm to (182.6, 110.0)
- moved SW1 4.65 mm to (167.0, 102.2), turned to 90 degrees
- moved R20 3.79 mm to (139.8, 99.8), turned to 90 degrees
- moved R22 3.75 mm to (139.8, 96.6), turned to -90 degrees
- moved R4 3.53 mm to (164.1, 90.1), turned to -90 degrees
- moved C30 2.89 mm to (145.0, 105.7)
- moved C2 2.51 mm to (148.9, 83.2)
- moved C3 2.51 mm to (150.6, 83.2)
- moved FB1 2.51 mm to (147.2, 83.2)
- moved C26 2.42 mm to (141.2, 103.1)
- renumbered C8 to C10, C9 to C11, C10 to C12, C11 to C13, C12 to C14, C13 to C15, C14 to C16, C15 to C17, C17 to C18, C18 to C19, C33 to C2, C19 to C20, C20 to C21, C21 to C22, C22 to C23, C23 to C24, C32 to C3, C28 to C30, C29 to C32, C25 to C33, C30 to C34, C31 to C35, C2 to C4, C3 to C5, C4 to C6, C5 to C7, C7 to C9, SW2 to SW3
Connections:
- C27 pad 1: VDC -> GND
- C27 pad 2: GND -> /VREF+
- J2 pad A6: Net-(J2-D+-PadA6) -> unconnected-(J2-D+-PadA6)
- J2 pad A7: Net-(J2-D--PadA7) -> unconnected-(J2-D--PadA7)
- J2 pad B6: Net-(J2-D+-PadA6) -> unconnected-(J2-D+-PadB6)
- J2 pad B7: Net-(J2-D--PadA7) -> unconnected-(J2-D--PadB7)
- U4 pad 20: unconnected-(U4-VREF+-Pad20) -> /VREF+
- U4 pad 42: unconnected-(U4-PB5-Pad42) -> /UCPD_DB
- U4 pad 5: Net-(U4-PF0) -> unconnected-(U4-PF0-Pad5)
- U5 pad 10: +3V3 -> /UCPD_DB
- U7 pad 1: GND -> Net-(J3-D--PadA7)
- U7 pad 2: +3V3 -> GND
- U7 pad 3: VDC -> Net-(J3-D+-PadA6)
Routing:
- net /UCPD_DB: track 0.00 -> 32.5 mm, vias 0 -> 2
- net Net-(U7-VBUS): track 0.00 -> 14.5 mm
- net /NRST: track 40.6 -> 31.6 mm
- net Net-(J3-D--PadA7): track 0.00 -> 7.26 mm
- net +3V3: track 73.4 -> 67.1 mm, vias 28 -> 27
- net Net-(J3-D+-PadA6): track 0.00 -> 5.87 mm
- net GND: track 10.6 -> 16.5 mm
- net Net-(J2-D--PadA7): track 5.54 -> 0.00 mm
- net /ADC1_IN4: track 41.6 -> 46.9 mm
- net /VREF+: track 0.00 -> 4.83 mm
- net /_USB_D_P: track 38.1 -> 33.8 mm
- net Net-(J2-D+-PadA6): track 4.34 -> 0.00 mm
- net Net-(U10-SW): track 0.00 -> 3.53 mm
- net /CC1: track 24.6 -> 21.1 mm
- net /_USB_D_N: track 36.2 -> 33.4 mm
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Other:
- board text added: "af 24 v6 rev b"
- board text removed: "af 24 rev a"

Commit message: chore: clean up submodules
Parts:
- added C29: 10u, Capacitor_SMD:C_1206_3216Metric, F.Cu at (99.6, 102.4)
- added C8: 10u, Capacitor_SMD:C_1206_3216Metric, F.Cu at (99.6, 99.9)
- added D8: B5819W SL, Diode_SMD:D_SOD-123, F.Cu at (142.5, 102.6)
- added D9: B5819W SL, Diode_SMD:D_SOD-123, F.Cu at (139.2, 105.1)
- added L2: 10u, Inductor_SMD:L_Abracon_ASPI-0630LR, F.Cu at (99.2, 94.1)
- C33: value 100n -> DNP
- J2: value USB_C_Receptacle_USB2.0_16P -> POWER
- J3: value USB_C_Receptacle_USB2.0_16P -> DEBUG
- moved C26 6.75 mm to (134.5, 103.0), turned to -90 degrees
- moved C30 1.93 mm to (144.1, 107.4)
- moved C31 1.93 mm to (146.6, 107.4)
- moved L1 1.93 mm to (143.6, 112.2)
- moved U10 1.93 mm to (140.9, 108.0)
Connections:
- net Net-(U7-VBUS) renamed +5VP
- D6 pad 1: /HEATER -> Net-(D6-K)
- Q3 pad 5: /HEATER -> Net-(D6-K)
- Q3 pad 6: /HEATER -> Net-(D6-K)
- Q3 pad 7: /HEATER -> Net-(D6-K)
- Q3 pad 8: /HEATER -> Net-(D6-K)
- U10 pad 2: VDC -> Net-(D8-K)
- U10 pad 3: VDC -> Net-(D8-K)
Routing:
- net +5VP: track 14.5 -> 75.6 mm
- net Net-(D8-K): track 0.00 -> 4.90 mm
- net VDC: track 49.1 -> 45.6 mm
- net GND: track 16.5 -> 14.4 mm
Other:
- board size 80 x 50.5 mm -> 91.5 x 50.5 mm

Commit message: fix: working revision
Parts:
- removed C29, C8: 10u, Capacitor_SMD:C_1206_3216Metric
- removed L2: 10u, Inductor_SMD:L_Abracon_ASPI-0630LR
Connections:
- D6 pad 1: Net-(D6-K) -> /HEATER
- Q3 pad 5: Net-(D6-K) -> /HEATER
- Q3 pad 6: Net-(D6-K) -> /HEATER
- Q3 pad 7: Net-(D6-K) -> /HEATER
- Q3 pad 8: Net-(D6-K) -> /HEATER

Commit message: chore: update PCB design
Parts:
- removed D3: BAT54S, Package_TO_SOT_SMD:SOT-23
- removed R10, R8: 10k, Resistor_SMD:R_0603_1608Metric
- removed TP1: 1C, Connector_Wire:SolderWire-0.75sqmm_1x01_D1.25mm_OD2.3mm
- removed TP2: 3P, Connector_Wire:SolderWire-0.75sqmm_1x01_D1.25mm_OD2.3mm
- removed TP3: 2T, Connector_Wire:SolderWire-0.75sqmm_1x01_D1.25mm_OD2.3mm
- removed TP4: 4D, Connector_Wire:SolderWire-0.75sqmm_1x01_D1.25mm_OD2.3mm
- removed TP5: 5S, Connector_Wire:SolderWire-0.75sqmm_1x01_D1.25mm_OD2.3mm
- added J4: XLR4, custom:MiniXLR-4_Switchcraft_TRAPCS_Horizontal, F.Cu at (113.1, 84.9)
- moved C33 14.3 mm to (119.1, 78.8)
- moved D7 14.3 mm to (122.7, 79.8)
- moved R25 14.3 mm to (119.1, 82.0)
- moved R26 14.3 mm to (119.1, 80.4)
- moved R28 7.22 mm to (129.9, 83.5), turned to -90 degrees
- moved U8 7.08 mm to (127.1, 80.8), turned to -90 degrees
- moved R9 6.81 mm to (119.1, 83.8), turned to 180 degrees
- moved R11 6.15 mm to (119.1, 85.5), turned to 0 degrees
- moved D6 4.69 mm to (111.1, 93.9)
- moved C32 3.25 mm to (129.9, 80.2), turned to -90 degrees
- moved R27 2.16 mm to (131.6, 80.2), turned to -90 degrees
- moved D4 1.90 mm to (122.7, 84.7), turned to 180 degrees
Connections:
- U4 pad 22: /_SLEEP -> unconnected-(U4-PB10-Pad22)
Routing:
- net /_SLEEP: track 30.6 -> 0.00 mm, vias 2 -> 0
- net /SLEEP: track 3.68 -> 0.00 mm
- net +3V3: track 67.1 -> 63.8 mm, vias 27 -> 26
- net /ADC2_IN2: track 45.4 -> 48.5 mm
- net /DET: track 3.70 -> 6.72 mm
- net Net-(D7-COM): track 5.37 -> 8.20 mm
- net /ADC2_IN1: track 40.1 -> 42.0 mm
- net /TC+: track 8.43 -> 7.11 mm
- net GND: vias 53 -> 52
Other:
- board size 91.5 x 50.5 mm -> 80 x 50.5 mm

Commit message: chore: generate production outputs
Parts:
- C27: renamed from C33; value DNP -> ~
- U7: renamed from U8; footprint Package_TO_SOT_SMD:SOT-23-5 -> Package_TO_SOT_SMD:SOT-23-5_HandSoldering
- moved J1 0.09 mm to (175.6, 109.0)
- renumbered C11 to C10, C12 to C11, C27 to C12, C28 to C13, C16 to C14, C17 to C15, C18 to C16, C19 to C17, C13 to C18, C14 to C19, C4 to C2, C25 to C23, C26 to C24, C15 to C25, C32 to C26, C23 to C28, C24 to C29, C5 to C3, C34 to C30, C35 to C31, C30 to C32, C31 to C33, C6 to C4, C7 to C5, C2 to C6, C3 to C7, C9 to C8, C10 to C9, D4 to D1, D1 to D2, D2 to D3, D6 to D4, D7 to D5, D5 to D6, D9 to D7, J3 to J2, J2 to J3, R33 to R1, R15 to R10, R16 to R11, R17 to R12, R18 to R13, R19 to R14, R7 to R15, R21 to R16, R12 to R17, R23 to R18, R13 to R19, R34 to R2, R24 to R20, R25 to R21, R26 to R22, R27 to R23, R20 to R24, R28 to R25, R22 to R26, R29 to R27, R30 to R28, R31 to R29, R32 to R30, R9 to R7, R11 to R8, R14 to R9, SW3 to SW2, U7 to U1, U9 to U8, U10 to U9
Routing:
- net GND: track 14.4 -> 17.0 mm
Other:
- board text removed: "*"

Commit message: fix: hardware issues
Parts:
- removed D5: BAT54S, Package_TO_SOT_SMD:SOT-23
- J4: value XLR4 -> TRAPC4MSX
- L1: value 10u -> LMDND4040WKT100MM
- U7: footprint Package_TO_SOT_SMD:SOT-23-5_HandSoldering -> Package_TO_SOT_SMD:SOT-23-5
Connections:
- J4 pad 1: /TC+ -> GND
- J4 pad 2: /DET -> /HEATER
- J4 pad 3: /HEATER -> /TC+
- J4 pad 4: GND -> /DET
Routing:
- net /TC+: track 7.11 -> 13.1 mm, vias 0 -> 1
- net /DET: track 6.51 -> 7.95 mm, vias 0 -> 1
- net +3V3: track 63.8 -> 62.7 mm, vias 26 -> 25
- net GND: track 17.0 -> 16.9 mm, vias 52 -> 51

Commit message: fix: pcb for minor mistakes
Parts:
- added C34: 10u, Capacitor_SMD:C_1206_3216Metric, F.Cu at (146.2, 101.5)
Routing:
- net GND: track 16.9 -> 18.3 mm, vias 51 -> 58
Other:
- board text added: "af 24 v6 rev c"
- board text removed: "af 24 v6 rev b"
