File: hardware/pcbs/ad_fs/ad_fs.kicad_pcb (KiCad board)
At the start: 2 copper layers, 30.1 x 11.9 mm, 3 parts, among them J1 XLR5, J2 XLR5, J3 Conn_01x03_Socket

Commit message: feat: hw v7a
Parts:
- added oshw1: Logo_Open_Hardware_Large, Symbol:OSHW-Symbol_6.7x6mm_SilkScreen, F.Cu at (146.0, 102.9)
- J3: value Conn_01x03_Socket -> SLP
- moved J3 7.00 mm to (147.0, 107.8)
Connections:
- net /GND renamed /BLUE
- net /HEATER renamed /RED
- J1 pad 2: /TC+ -> /SLP
- J1 pad 4: /SLP -> /GREEN
- J2 pad 2: /TC+ -> /SLP
- J2 pad 4: /SLP -> /GREEN
Routing:
- net /TC+: track 21.4 -> 0.00 mm
- net /GREEN: track 0.00 -> 20.5 mm
- net /SLP: track 20.1 -> 21.5 mm
- net /DET: track 21.0 -> 21.8 mm
Other:
- board text added: "af 25 v7a"
