File: hardware/pcbs/ad_fs/ad_fs.kicad_sch (KiCad schematic)
At the start: 3 parts, among them J1 XLR5, J2 XLR5, J3 Conn_01x03_Socket

Commit message: feat: hw v7a
Parts:
- added oshw1: Logo_Open_Hardware_Large, Symbol:OSHW-Symbol_6.7x6mm_SilkScreen, symbol Graphic:Logo_Open_Hardware_Large
- J3: value Conn_01x03_Socket -> SLP
Connections:
- net TC+ is gone; now on net SLP: J1.2 (P2), J2.2 (P2)
- net SLP: no longer J1.4 (P3), J2.4 (P3)
- net GND renamed BLUE
- net HEATER renamed RED
- new net GREEN: J1.4 (P3), J2.4 (P3)
Other:
- title: MiniXLR adapter -> MiniXLR adapter (AD-FS)
