File: hardware/pcbs/holder/holder.kicad_pcb (KiCad board)
At the start: 2 copper layers, 80 x 50.5 mm, 0 parts

Commit message: chore: finalize v6c production run
Other:
- outline, holes or cut-outs redrawn
